File: PCB/blackmacro_base/blackmacro_base.kicad_pcb (KiCad board)
At the start: 2 copper layers, 182.4 x 118.2 mm, 127 parts, among them J1 MOD Power, J2 MOD I/O, J3 Dial_PowerConn, J4 Dial_MagEncoderConn, J5 Dial_MotorControlConn, U2 74HC238, U3 SN74LVC1T45DBV

Commit message: updated pico footprint for pcb usb connections
Parts:
- A1: footprint Module:RaspberryPi_Pico_W_SMD_HandSolder -> pico:RaspberryPi_Pico_W_SMD_THTdebug
Connections:
- A1 pad D1: (no net) -> unconnected-(A1-SWCLK-PadD1)
- A1 pad D2: (no net) -> GND
- A1 pad D3: (no net) -> unconnected-(A1-SWDIO-PadD3)
Routing:
- net +3V3: track 252.2 -> 252.9 mm

Commit message: switched to pcb usb socket, battery management wip switched to pouch instead of 16850 pcb ready for rewiring + keyboard adjustments
Parts:
- removed H1, H2, H3, H4, H5, H6: MountingHole, MountingHole:MountingHole_3.2mm_M3_ISO14580_Pad
- added J6: USB_C_Receptacle_USB2.0_16P, Connector_USB:USB_C_Receptacle_HCTL_HC-TYPE-C-16P-01A, F.Cu at (152.0, 42.5)
- A1: footprint pico:RaspberryPi_Pico_W_SMD_THTdebug -> Module:RaspberryPi_Pico_W_SMD
- J3, J4, J5: moved to F.Cu
- U2: moved to B.Cu
- moved A1 51.4 mm to (149.6, 145.8)
- moved U2 50.1 mm to (149.4, 145.5)
- moved J4 13.7 mm to (186.0, 95.6), turned to 0 degrees
- moved J3 13.7 mm to (223.3, 96.0), turned to 180 degrees
- moved J5 12.2 mm to (167.1, 102.1), turned to -90 degrees
- moved C10 8.88 mm to (87.6, 164.8)
- moved C7 8.88 mm to (89.2, 131.3)
- moved D17 8.88 mm to (69.3, 154.7)
- moved D18 8.88 mm to (107.4, 154.7)
- moved LED15 8.88 mm to (98.8, 164.8)
- moved LED16 8.88 mm to (60.7, 164.8)
- moved SW_LD1 8.88 mm to (60.7, 140.7)
- moved SW_LD2 8.88 mm to (79.8, 140.7)
- moved SW_LD3 8.88 mm to (98.8, 140.7)
- moved SW_LD4 8.88 mm to (117.9, 140.7)
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Routing:
- net +3V3: track 252.9 -> 90.6 mm, vias 5 -> 3
- net Net-(LED16-DOUT): track 234.3 -> 79.2 mm, vias 2 -> 0
- net +5V: track 677.8 -> 538.4 mm, vias 26 -> 22
- net MT_COL1: track 215.4 -> 93.8 mm, vias 4 -> 1
- net SCL: track 118.2 -> 0.00 mm, vias 2 -> 0
- net SDA: track 114.6 -> 0.53 mm, vias 2 -> 0
- net MT_ROW5: track 240.8 -> 131.4 mm, vias 4 -> 3
- net MOD_IO: track 78.1 -> 3.88 mm, vias 3 -> 0
- net /RENC2_A: track 102.2 -> 33.7 mm, vias 3 -> 0
- net /RENC2_B: track 99.7 -> 31.4 mm, vias 3 -> 0
- net MT_ROW6: track 122.6 -> 60.8 mm
- net MT_COL4: track 238.4 -> 184.0 mm, vias 7 -> 6
- net /MAG_DO: track 49.0 -> 0.00 mm, vias 1 -> 0
- net MT_COL2: track 286.8 -> 239.2 mm, vias 7 -> 6
- net MT_COL3: track 217.3 -> 170.2 mm, vias 9 -> 6
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- removed copper zone on B.Cu, net GND
- removed copper zone on F.Cu, net GND
Other:
- board size 182.4 x 118.2 mm -> 182.6 x 132.4 mm
- board text removed: "5.1k Adapter ADHESIVE HERE"
- board text removed: "5.1k adapter cutout"
