File: PCB/blackmacro_base/blackmacro_base.kicad_pcb (KiCad board)
At the start: 2 copper layers, 182.6 x 132.4 mm, 122 parts, among them J1 MOD Power, J2 MOD I/O, J3 Dial_PowerConn, J4 Dial_MagEncoderConn, J5 Dial_MotorControlConn, J6 USB_C_Receptacle_USB2.0_16P, U2 74HC238, U3 SN74LVC1T45DBV

Commit message: schematics done, working on pcb
Parts:
- removed kibuzzard-6A2F9E22: G***, kibuzzard-6A2F9E22
- removed kibuzzard-6A2FA9CB: G***, kibuzzard-6A2FA9CB
- added BT1: FLY.906090.6000, Connector_JST:JST_EH_S3B-EH_1x03_P2.50mm_Horizontal, B.Cu at (111.0, 32.5)
- added C1: 10uF, Capacitor_SMD:C_0603_1608Metric_Pad1.08x0.95mm_HandSolder, F.Cu at (202.9, -3.56)
- added C13: 22uF, Capacitor_SMD:C_0603_1608Metric_Pad1.08x0.95mm_HandSolder, F.Cu at (203.6, 4.76)
- added C14: 0.1uF, Capacitor_SMD:C_1206_3216Metric_Pad1.33x1.80mm_HandSolder, F.Cu at (217.5, 18.7)
- added C15: 3.3uF, Capacitor_SMD:C_0603_1608Metric_Pad1.08x0.95mm_HandSolder, F.Cu at (203.6, 7.27)
- added C16: 3.3uF, Capacitor_SMD:C_0603_1608Metric_Pad1.08x0.95mm_HandSolder, F.Cu at (203.6, 9.78)
- added C17: 22uF, Capacitor_SMD:C_0603_1608Metric_Pad1.08x0.95mm_HandSolder, F.Cu at (203.6, 12.3)
- added C18: 0.1uF, Capacitor_SMD:C_1206_3216Metric_Pad1.33x1.80mm_HandSolder, F.Cu at (217.5, 22.0)
- added C19: 10uF, Capacitor_SMD:C_0603_1608Metric_Pad1.08x0.95mm_HandSolder, F.Cu at (203.6, 14.8)
- added C2: 10uF, Capacitor_SMD:C_0603_1608Metric_Pad1.08x0.95mm_HandSolder, F.Cu at (203.6, 2.25)
- added C20: 3.3uF, Capacitor_SMD:C_0603_1608Metric_Pad1.08x0.95mm_HandSolder, F.Cu at (208.0, -3.81)
- added C21: 10uF, Capacitor_SMD:C_0603_1608Metric_Pad1.08x0.95mm_HandSolder, F.Cu at (208.0, 2.25)
- added C22: 3.3uF, Capacitor_SMD:C_0603_1608Metric_Pad1.08x0.95mm_HandSolder, F.Cu at (208.0, 4.76)
- added C23: OPTIONAL, Capacitor_SMD:C_1206_3216Metric_Pad1.33x1.80mm_HandSolder, F.Cu at (217.5, 25.4)
- added C24: OPTIONAL, Capacitor_SMD:C_1206_3216Metric_Pad1.33x1.80mm_HandSolder, F.Cu at (217.5, 28.7)
- added C25: 10uF, Capacitor_SMD:C_0603_1608Metric_Pad1.08x0.95mm_HandSolder, F.Cu at (208.0, 7.27)
- added D25: SS54, Diode_SMD:D_SMA_Handsoldering, F.Cu at (231.6, 0.76)
- added D26: SS54_optional, Diode_SMD:D_SMA_Handsoldering, F.Cu at (257.6, 20.8)
- added DB1: STDBY, LED_SMD:LED_0603_1608Metric_Pad1.05x0.95mm_HandSolder, F.Cu at (210.8, 29.1)
- added DB2: Charge, LED_SMD:LED_0603_1608Metric_Pad1.05x0.95mm_HandSolder, F.Cu at (210.8, 31.7)
- added F1: hold=2, trip=3.5, Fuse:Fuse_1206_3216Metric_Pad1.42x1.75mm_HandSolder, F.Cu at (236.5, 15.3)
- added JP1: ChargeSigJumper, Jumper:SolderJumper-2_P1.3mm_Open_TrianglePad1.0x1.5mm, F.Cu at (222.7, 18.8)
- added JP2: Batt 5v no schottky, Jumper:SolderJumper-2_P1.3mm_Bridged_Pad1.0x1.5mm, F.Cu at (222.7, 22.3)
- added JP3: E1, Jumper:SolderJumper-2_P1.3mm_Bridged_RoundedPad1.0x1.5mm, F.Cu at (222.7, 25.9)
- added JP4: E2, Jumper:SolderJumper-2_P1.3mm_Bridged_RoundedPad1.0x1.5mm, F.Cu at (222.7, 29.4)
- added JP5: E3, Jumper:SolderJumper-2_P1.3mm_Bridged_RoundedPad1.0x1.5mm, F.Cu at (222.7, 33.0)
- added L1: 4.7uH, Inductor_SMD:L_Changjiang_FXL0630, F.Cu at (219.5, 12.9)
- added Q1: AO3415, Package_TO_SOT_SMD:SOT-23_Handsoldering, F.Cu at (238.0, 29.2)
- added Q2: AO3415, Package_TO_SOT_SMD:SOT-23_Handsoldering, F.Cu at (238.0, 33.9)
- added R1: 0.4, Resistor_SMD:R_2512_6332Metric_Pad1.40x3.35mm_HandSolder, F.Cu at (229.0, 11.3)
- added R10: 5.1k, Resistor_SMD:R_0603_1608Metric_Pad0.98x0.95mm_HandSolder, F.Cu at (208.0, 14.8)
- added R11: 5.1k, Resistor_SMD:R_0603_1608Metric_Pad0.98x0.95mm_HandSolder, F.Cu at (212.3, -0.26)
- added R12: 8.2k, Resistor_SMD:R_0805_2012Metric_Pad1.20x1.40mm_HandSolder, F.Cu at (210.9, 23.4)
- added R13: 8.2k, Resistor_SMD:R_0805_2012Metric_Pad1.20x1.40mm_HandSolder, F.Cu at (210.9, 26.4)
- added R14: 5.1k, Resistor_SMD:R_0603_1608Metric_Pad0.98x0.95mm_HandSolder, F.Cu at (212.3, 2.25)
- added R15: 37.4k, Resistor_SMD:R_0603_1608Metric_Pad0.98x0.95mm_HandSolder, F.Cu at (212.3, 4.76)
- added R16: 100k, Resistor_SMD:R_0603_1608Metric_Pad0.98x0.95mm_HandSolder, F.Cu at (212.3, 7.27)
- added R2: 150, Resistor_SMD:R_0603_1608Metric_Pad0.98x0.95mm_HandSolder, F.Cu at (208.0, 9.78)
- added R3: 150, Resistor_SMD:R_0603_1608Metric_Pad0.98x0.95mm_HandSolder, F.Cu at (208.0, 12.3)
- added R4: 1.2k, Resistor_SMD:R_0805_2012Metric_Pad1.20x1.40mm_HandSolder, F.Cu at (210.9, 17.5)
- added R9: 1.2k, Resistor_SMD:R_0805_2012Metric_Pad1.20x1.40mm_HandSolder, F.Cu at (210.9, 20.5)
- added SW1: SW_SPDT, Button_Switch_SMD:SW_SPDT_Shouhan_MSK12C02, F.Cu at (144.0, 42.7)
- added TH1: 10k, 43C=4.791k, Connector_Wire:SolderWire-0.127sqmm_1x02_P3.7mm_D0.48mm_OD1mm_Relief, F.Cu at (120.1, 70.9)
- added TP10: VBAT, TestPoint:TestPoint_THTPad_D1.5mm_Drill0.7mm, F.Cu at (206.8, 24.9)
- added TP11: FB, TestPoint:TestPoint_Pad_D1.0mm, F.Cu at (210.1, 34.6)
- added TP12: 5V, TestPoint:TestPoint_THTPad_D1.5mm_Drill0.7mm, F.Cu at (206.8, 28.5)
- added TP14: VBUS, TestPoint:TestPoint_THTPad_D1.5mm_Drill0.7mm, F.Cu at (206.8, 32.0)
- added TP3: USB+, TestPoint:TestPoint_Pad_D1.5mm, F.Cu at (203.2, 17.8)
- added TP4: USB-, TestPoint:TestPoint_Pad_D1.5mm, F.Cu at (203.2, 21.4)
- added TP5: CHRG, TestPoint:TestPoint_Pad_D1.5mm, F.Cu at (203.2, 24.9)
- added TP6: STDBY, TestPoint:TestPoint_Pad_D1.5mm, F.Cu at (203.2, 28.5)
- added TP7: SRX, TestPoint:TestPoint_THTPad_D1.5mm_Drill0.7mm, F.Cu at (203.2, 32.0)
- added TP8: BAT, TestPoint:TestPoint_THTPad_D1.5mm_Drill0.7mm, F.Cu at (206.8, 17.8)
- added TP9: TEMP, TestPoint:TestPoint_Pad_D1.5mm, F.Cu at (206.8, 21.4)
- added U1: HTP4056-42-ESOP8, Package_SO:SOIC-8-1EP_3.9x4.9mm_P1.27mm_EP2.41x3.3mm_ThermalVias, F.Cu at (236.5, 20.4)
- added U4: BQ27427, Package_BGA:Texas_DSBGA-9_1.62x1.58mm_Layout3x3_P0.5mm, F.Cu at (217.9, 39.9)
- added U5: MT3608L, Package_TO_SOT_SMD:SOT-23-6_Handsoldering, F.Cu at (236.4, 11.3)
- A1: footprint Module:RaspberryPi_Pico_W_SMD -> pico:RaspberryPi_Pico_W_SMD_THTdebug
- J2: footprint Connector_PinSocket_2.54mm:PinSocket_1x03_P2.54mm_Horizontal -> Connector_PinSocket_2.54mm:PinSocket_1x02_P2.54mm_Horizontal
- J5: moved to B.Cu
- TP13: renamed from TP_KROW1; value TestPoint -> KROW1; footprint TestPoint:TestPoint_THTPad_D1.5mm_Drill0.7mm -> TestPoint:TestPoint_Pad_D1.0mm
- TP15: renamed from TP_KROW2; value TestPoint -> KROW2; footprint TestPoint:TestPoint_THTPad_D1.5mm_Drill0.7mm -> TestPoint:TestPoint_Pad_D1.0mm
- TP16: renamed from TP_VBUS1; value VSYS test point -> VSYS
- TP17: renamed from TP_3V1; value VSYS test point -> 3V3
- TP18: renamed from TP_KROW3; value TestPoint -> KROW3; footprint TestPoint:TestPoint_THTPad_D1.5mm_Drill0.7mm -> TestPoint:TestPoint_Pad_D1.0mm
- TP19: renamed from TP_KROW4; value TestPoint -> KROW4; footprint TestPoint:TestPoint_THTPad_D1.5mm_Drill0.7mm -> TestPoint:TestPoint_Pad_D1.0mm
- TP20: renamed from TP_KROW5; value TestPoint -> KROW5; footprint TestPoint:TestPoint_THTPad_D1.5mm_Drill0.7mm -> TestPoint:TestPoint_Pad_D1.0mm
- TP21: renamed from TP_GND1; value VSYS test point -> GND
- TP22: renamed from TP_KROW6; value TestPoint -> KROW6; footprint TestPoint:TestPoint_THTPad_D1.5mm_Drill0.7mm -> TestPoint:TestPoint_Pad_D1.0mm
- TP23: renamed from TP_KCOL1; value TestPoint -> KCOL1; footprint TestPoint:TestPoint_THTPad_D1.5mm_Drill0.7mm -> TestPoint:TestPoint_Pad_D1.0mm
- TP24: renamed from TP_KCOL2; value TestPoint -> KCOL2; footprint TestPoint:TestPoint_THTPad_D1.5mm_Drill0.7mm -> TestPoint:TestPoint_Pad_D1.0mm
- TP25: renamed from TP_KCOL3; value TestPoint -> KCOL3; footprint TestPoint:TestPoint_THTPad_D1.5mm_Drill0.7mm -> TestPoint:TestPoint_Pad_D1.0mm
- TP26: renamed from TP_KCOL4; value TestPoint -> KCOL4; footprint TestPoint:TestPoint_THTPad_D1.5mm_Drill0.7mm -> TestPoint:TestPoint_Pad_D1.0mm
- TP_LED1, TP_LED2: footprint TestPoint:TestPoint_THTPad_D1.5mm_Drill0.7mm -> TestPoint:TestPoint_Pad_D1.5mm
- moved G*** 113.2 mm to (26.7, 86.4)
- moved TP23 83.8 mm to (157.7, 18.3)
- moved TP25 77.6 mm to (165.9, 19.8)
- moved G*** 77.5 mm to (129.8, 163.6)
- moved TP24 76.1 mm to (129.0, 29.7)
- moved kibuzzard-6A2FA9C2 69.4 mm to (149.6, 145.8)
- moved TP13 64.5 mm to (142.0, 19.3)
- moved J5 42.0 mm to (130.0, 121.8)
- moved U2 16.4 mm to (132.9, 145.4)
- moved TP16 11.1 mm to (157.0, 64.3)
- moved J3 9.47 mm to (213.8, 96.8)
- moved TP1 8.18 mm to (141.5, 60.7)
- moved J2 2.77 mm to (135.4, 55.2)
- moved J6 2.06 mm to (153.9, 43.3)
- moved J4 1.36 mm to (185.4, 96.8)
Connections:
- A1 pad 25: MOD_IO -> CHRG
- A1 pad 39: unconnected-(A1-VSYS-Pad39) -> BAT_VSYS
- A1 pad TP1: unconnected-(A1-USB_GND-PadTP1) -> GND
- A1 pad TP2: unconnected-(A1-USB_DM-PadTP2) -> USB_D-
- A1 pad TP3: unconnected-(A1-USB_DP-PadTP3) -> USB_D+
- J2 pad 1: MOD_IO -> MOD_O1
- J2 pad 2: MOD_O1 -> MOD_O2
- J3 pad 1: +3V3 -> GND
- J3 pad 3: GND -> +3V3
- J4 pad 1: unconnected-(J4-Pin_1-Pad1) -> /MAG_PUSH
- J4 pad 2: unconnected-(J4-Pin_2-Pad2) -> /MAG_OUT
- J4 pad 3: unconnected-(J4-Pin_3-Pad3) -> /MAG_CSN
- J4 pad 4: /MAG_DO -> /MAG_CLK
- J4 pad 5: /MAG_CLK -> /MAG_DO
- J4 pad 6: /MAG_CSN -> unconnected-(J4-Pin_6-Pad6)
- J4 pad 7: /MAG_OUT -> unconnected-(J4-Pin_7-Pad7)
- J4 pad 8: /MAG_PUSH -> unconnected-(J4-Pin_8-Pad8)
- J6 pad A1: Net-(J6-GND-PadA1) -> GND
- J6 pad A12: Net-(J6-GND-PadA1) -> GND
- J6 pad A5: unconnected-(J6-CC1-PadA5) -> Net-(J6-CC1)
- J6 pad A6: unconnected-(J6-D+-PadA6) -> USB_D+
- J6 pad A7: unconnected-(J6-D--PadA7) -> USB_D-
- J6 pad B1: Net-(J6-GND-PadA1) -> GND
- J6 pad B12: Net-(J6-GND-PadA1) -> GND
- J6 pad B5: unconnected-(J6-CC2-PadB5) -> Net-(J6-CC2)
- J6 pad B6: unconnected-(J6-D+-PadB6) -> USB_D+
- J6 pad B7: unconnected-(J6-D--PadB7) -> USB_D-
- J6 pad SH: unconnected-(J6-SHIELD-PadSH) -> GND
- TP16 pad 1: +5V -> BAT_VSYS
- U2 pad 10: MOD_O2 -> MT_ROW6
- U2 pad 11: MT_ROW1 -> MT_ROW5
- U2 pad 12: MT_ROW2 -> MT_ROW4
- U2 pad 14: MT_ROW4 -> MT_ROW2
- U2 pad 15: MT_ROW5 -> MT_ROW1
- U2 pad 4: GND -> Net-(JP3-B)
- U2 pad 5: GND -> Net-(JP4-B)
- U2 pad 6: +3V3 -> Net-(JP5-B)
- U2 pad 7: MT_ROW6 -> MOD_O2
Routing:
- net MT_COL2: track 239.2 -> 157.0 mm, vias 6 -> 4
- net +3V3: track 90.6 -> 22.2 mm, vias 3 -> 2
- net MOD_O2: track 42.3 -> 0.00 mm
- net MOD_O1: track 39.9 -> 0.00 mm
- net MT_ROW1: track 105.2 -> 65.3 mm
- net /RENC2_B: track 31.4 -> 12.4 mm
- net /RENC2_A: track 33.7 -> 14.7 mm
- net MT_COL3: track 170.2 -> 153.1 mm
- net GND: track 9.87 -> 0.00 mm
- net MT_ROW3: track 75.9 -> 70.0 mm
- net Net-(D8-K): track 7.89 -> 3.06 mm
- net MOD_IO: track 3.88 -> 0.00 mm
Other:
- board size 182.6 x 132.4 mm -> 182.6 x 130.9 mm
- board text added: "0"
- board text added: "3.3"
- board text added: "5"
- board text added: "A"
- board text added: "B"
- board text added: "CLK"
- board text added: "CS"
- board text added: "DO"
- board text added: "PSH"
- board text added: "SIG"
- board text added: "UH"
- board text added: "VERSION 2"
- board text added: "Z"
- board text removed: "Version 1"

Commit message: everything routed except led
Parts:
- removed JP2: Batt 5v no schottky, Jumper:SolderJumper-2_P1.3mm_Bridged_Pad1.0x1.5mm
- added D27: SS54, Diode_SMD:D_SMA_Handsoldering, F.Cu at (155.8, 97.8)
- added Q3: AO3415, Package_TO_SOT_SMD:SOT-23_Handsoldering, F.Cu at (141.2, 71.0)
- C25, R5, R6, R7, R8: moved to B.Cu
- C4, C5, U2, U3: moved to F.Cu
- TP27: renamed from TP_LED1; value TestPoint -> LED1
- TP28: renamed from TP_LED2; value TestPoint -> LED2
- moved TP27 167.1 mm to (195.0, -71.2)
- moved TP21 163.2 mm to (171.8, -44.6)
- moved TP18 158.8 mm to (166.0, -38.5)
- moved TP19 147.4 mm to (165.8, 9.50)
- moved TP17 145.4 mm to (167.9, -28.3)
- moved TP28 139.4 mm to (185.1, -35.9)
- moved TP15 138.7 mm to (188.8, -29.8)
- moved C22 132.5 mm to (163.4, 129.5)
- moved C25 128.5 mm to (154.8, 124.2), turned to 180 degrees
- moved TP22 128.4 mm to (181.5, -31.0)
- moved TP2 124.3 mm to (160.4, -58.9)
- moved TP1 123.8 mm to (155.2, -62.3)
- moved D26 123.6 mm to (160.8, 97.8), turned to 90 degrees
- moved U1 121.5 mm to (139.3, 93.3), turned to 180 degrees
- moved JP1 121.1 mm to (133.8, 101.0), turned to -90 degrees
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Connections:
- A1 pad 10: /MOTR_WH -> /MOTR_UL
- A1 pad 11: /MOTR_VL -> /MOTR_VH
- A1 pad 12: /MOTR_VH -> /MOTR_VL
- A1 pad 14: /MOTR_UL -> /MOTR_WH
- A1 pad 15: /MOTR_UH -> /MOTR_WL
- A1 pad 40: +5V -> VBUS
- A1 pad 9: /MOTR_WL -> /MOTR_UH
- C14 pad 2: VBAT -> Net-(Q3-G)
- C18 pad 2: +5V -> VBUS
- C21 pad 1: +5V -> VBUS
- F1 pad 2: +5V -> VBUS
- J1 pad 1: +3V3 -> GND
- J1 pad 2: +5V -> +3V3
- J1 pad 3: GND -> +5V
- Q1 pad 1: +5V -> VBUS
- Q1 pad 2: BAT_VSYS -> VBAT
- Q1 pad 3: VBAT -> BAT_VSYS
- Q2 pad 1: +5V -> VBUS
- R1 pad 1: +5V -> VBUS
- R16 pad 1: +5V -> VBUS
- SW1 pad 1: VBAT -> /SRX
- SW1 pad 2: /SRX -> Net-(Q3-G)
- SW1 pad 3: unconnected-(SW1-C-Pad3) -> GND
- TP14 pad 1: +5V -> VBUS
- TP5 pad 1: Net-(DB2-A) -> Net-(DB2-K)
- TP6 pad 1: Net-(DB1-A) -> Net-(DB1-K)
- U2 pad 10: MT_ROW6 -> MT_ROW1
- U2 pad 11: MT_ROW5 -> MT_ROW2
- U2 pad 12: MT_ROW4 -> MT_ROW3
- U2 pad 13: MT_ROW3 -> MT_ROW4
- U2 pad 14: MT_ROW2 -> MT_ROW5
- U2 pad 15: MT_ROW1 -> MT_ROW6
Routing:
- net /RENC2_B: track 12.4 -> 278.0 mm, vias 0 -> 2
- net +3V3: track 22.2 -> 287.1 mm, vias 2 -> 6
- net /RENC2_A: track 14.7 -> 272.1 mm
- net MT_ROW5: track 131.4 -> 291.2 mm, vias 3 -> 7
- net Net-(LED16-DOUT): track 79.2 -> 233.1 mm, vias 0 -> 4
- net +5V: track 538.4 -> 686.1 mm, vias 22 -> 24
- net SCL: track 0.00 -> 145.7 mm, vias 0 -> 3
- net SDA: track 0.53 -> 143.4 mm, vias 0 -> 3
- net MT_COL2: track 157.0 -> 296.8 mm, vias 4 -> 9
- net MT_COL3: track 153.1 -> 280.9 mm, vias 6 -> 9
- net VBUS: track 0.00 -> 104.5 mm
- net /MAG_DO: track 0.00 -> 99.0 mm, vias 0 -> 1
- net /MAG_CSN: track 0.00 -> 94.9 mm, vias 0 -> 1
- net /MAG_CLK: track 0.00 -> 91.7 mm, vias 0 -> 1
- net /SRX: track 0.00 -> 88.8 mm, vias 0 -> 2
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- added copper zone on B.Cu, net GND
- added copper zone on F.Cu, net GND
Other:
- outline, holes or cut-outs redrawn
- board text added: "+"
- board text added: "-"
- board text added: "3"
- board text added: "ANTENNA KEEPOUT"
- board text added: "CHRG SIG"
- board text added: "DEBUG"
- board text added: "EMF+HOT!"
- board text added: "FILL WITH LOTS OF SOLDER"
- board text added: "HOT!"
- board text added: "MAGENC"
- board text added: "MOD PWR"
- board text added: "MOTOR"
- board text added: "OPT"
- board text added: "PWR"
- board text added: "USB"
- board text added: "VIO"
- board text removed: "3V3"
- board text removed: "DIAG"
- board text removed: "MOD POWER"
- board text removed: "MagEnc"
- board text removed: "Motor"
- board text removed: "Power"
- board text removed: "SCL"
- board text removed: "SDA"
