File: PCB/blackmacro_base/blackmacro_base.kicad_pcb (KiCad board)
At the start: 2 copper layers, 182.6 x 130.9 mm, 178 parts, among them J1 MOD Power, J2 MOD I/O, J3 Dial_PowerConn, J4 Dial_MagEncoderConn, J5 Dial_MotorControlConn, J6 USB_C_Receptacle_USB2.0_16P, Q1 AO3415, Q2 AO3415, Q3 AO3415, SW1 SW_SPDT, U1 HTP4056-42-ESOP8, U2 74HC238, U3 SN74LVC1T45DBV, U4 BQ27427, U5 MT3608L

Commit message: before ground pour
Parts:
- TP16: footprint TestPoint:TestPoint_THTPad_D1.5mm_Drill0.7mm -> TestPoint:TestPoint_Pad_D1.5mm
- moved TP20 240.7 mm to (73.2, 162.6)
- moved TP18 194.8 mm to (70.1, 131.1)
- moved TP15 184.7 mm to (70.1, 111.8)
- moved TP19 170.1 mm to (70.1, 150.1)
- moved C5 168.0 mm to (94.0, 65.8), turned to 0 degrees
- moved TP23 167.9 mm to (66.5, 69.1), turned to 180 degrees
- moved TP16 166.6 mm to (163.6, 115.3), turned to 180 degrees
- moved C4 164.4 mm to (94.0, 68.6), turned to 0 degrees
- moved U3 163.0 mm to (100.5, 67.1), turned to 180 degrees
- moved TP27 161.5 mm to (105.2, 63.0), turned to 180 degrees
- moved TP13 153.8 mm to (72.6, 65.5), turned to 180 degrees
- moved TP2 148.7 mm to (82.5, 67.8), turned to 180 degrees
- moved TP25 148.5 mm to (101.6, 71.6)
- moved TP21 147.3 mm to (222.5, 93.7)
- moved TP1 147.2 mm to (86.4, 67.8), turned to 180 degrees
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Routing:
- net /LED_IN: track 0.00 -> 125.3 mm, vias 0 -> 2
- net MT_ROW6: track 60.8 -> 179.7 mm, vias 1 -> 8
- net MT_COL1: track 155.7 -> 262.6 mm, vias 2 -> 5
- net Net-(LED1-DIN): track 15.3 -> 43.6 mm, vias 0 -> 1
- net +5V: track 686.1 -> 714.0 mm
- net +3V3: track 287.1 -> 311.2 mm
- net Net-(U1-TEMP): track 44.0 -> 62.3 mm
- net MT_COL3: track 280.9 -> 290.6 mm
- net SCL: track 145.7 -> 153.2 mm
- net MT_ROW4: track 94.6 -> 101.8 mm
- net MT_ROW3: track 77.8 -> 85.0 mm
- net MT_ROW2: track 65.7 -> 72.6 mm
- net MT_ROW1: track 143.1 -> 149.6 mm
- net SDA: track 143.4 -> 149.9 mm
- net MT_COL4: track 258.1 -> 264.5 mm
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
Commit message: copper done todo: silkscreen + art
Parts:
- added REF**: Fiducial_0.5mm_Mask1mm, Fiducial:Fiducial_0.5mm_Mask1mm, F.Cu at (122.7, 151.9)
- added REF**: Fiducial_0.5mm_Mask1mm, Fiducial:Fiducial_0.5mm_Mask1mm, F.Cu at (174.2, 46.2)
- added REF**: Fiducial_0.5mm_Mask1mm, Fiducial:Fiducial_0.5mm_Mask1mm, F.Cu at (56.6, 62.0)
- added REF**: Fiducial_0.5mm_Mask1mm, Fiducial:Fiducial_0.5mm_Mask1mm, F.Cu at (223.5, 102.1)
- added REF**: Fiducial_0.5mm_Mask1mm, Fiducial:Fiducial_0.5mm_Mask1mm, B.Cu at (226.8, 49.5)
- added REF**: Fiducial_0.5mm_Mask1mm, Fiducial:Fiducial_0.5mm_Mask1mm, B.Cu at (57.9, 66.8)
- added REF**: Fiducial_0.5mm_Mask1mm, Fiducial:Fiducial_0.5mm_Mask1mm, B.Cu at (141.0, 62.2)
- added REF**: Fiducial_0.5mm_Mask1mm, Fiducial:Fiducial_0.5mm_Mask1mm, B.Cu at (166.9, 168.7)
- moved R10 0.80 mm to (149.5, 49.8)
- moved R11 0.80 mm to (149.5, 51.6)
Routing:
- net GND: track 9.45 -> 54.5 mm, vias 58 -> 244
- net Net-(J6-CC1): track 7.82 -> 9.07 mm
- net /MAG_DO: track 99.0 -> 100.2 mm
- net /MAG_CLK: track 91.7 -> 92.8 mm
Other:
- board text added: "ATLS-KIP-BMCR-BS-2-WLB"
- board text added: "BATTERY HERE"
- board text added: "I swear to god if the battery management fucks up the signals"
- board text added: "Remeber to tape the thermister onto the battery!"
- board text removed: "ATLS-KIP-BMCR-BS-1-WNB"
