File: PCB/blackmacro_base/blackmacro_base.kicad_sch (KiCad schematic)
At the start: 145 parts, among them J1 MOD Power, J2 MOD I/O, J3 Dial_PowerConn, J4 Dial_MagEncoderConn, J5 Dial_MotorControlConn, J6 USB_C_Receptacle_USB2.0_16P, Q1 AO3415, Q2 AO3415, SW1 SW_SPDT, U1 HTP4056-42-ESOP8, U2 74HC238, U3 SN74LVC1T45DBV, U4 BQ27427, U5 MT3608L

Commit message: schematics done, working on pcb
Parts:
- added C19, C21, C25: 10uF, Capacitor_SMD:C_0603_1608Metric_Pad1.08x0.95mm_HandSolder, symbol Device:C_Small
- added C20, C22: 3.3uF, Capacitor_SMD:C_0603_1608Metric_Pad1.08x0.95mm_HandSolder, symbol Device:C_Small
- added C23, C24: OPTIONAL, Capacitor_SMD:C_1206_3216Metric_Pad1.33x1.80mm_HandSolder, symbol Device:C_Small
- added D25: SS54, Diode_SMD:D_SMA_Handsoldering, symbol Device:D_Schottky
- added D26: SS54_optional, Diode_SMD:D_SMA_Handsoldering, symbol Device:D_Schottky
- added F1: hold=2, trip=3.5, Fuse:Fuse_1206_3216Metric_Pad1.42x1.75mm_HandSolder, symbol Device:Polyfuse
- added JP2: Batt 5v no schottky, Jumper:SolderJumper-2_P1.3mm_Bridged_Pad1.0x1.5mm, symbol Jumper:SolderJumper_2_Bridged
- added JP3: E1, Jumper:SolderJumper-2_P1.3mm_Bridged_RoundedPad1.0x1.5mm, symbol Jumper:SolderJumper_2_Bridged
- added JP4: E2, Jumper:SolderJumper-2_P1.3mm_Bridged_RoundedPad1.0x1.5mm, symbol Jumper:SolderJumper_2_Bridged
- added JP5: E3, Jumper:SolderJumper-2_P1.3mm_Bridged_RoundedPad1.0x1.5mm, symbol Jumper:SolderJumper_2_Bridged
- added R16: 100k, Resistor_SMD:R_0603_1608Metric_Pad0.98x0.95mm_HandSolder, symbol Device:R_Small
- added TP10: VBAT, TestPoint:TestPoint_THTPad_D1.5mm_Drill0.7mm, symbol Connector:TestPoint
- added TP11: FB, TestPoint:TestPoint_Pad_D1.0mm, symbol Connector:TestPoint
- added TP12: 5V, TestPoint:TestPoint_THTPad_D1.5mm_Drill0.7mm, symbol Connector:TestPoint
- added TP3: USB+, TestPoint:TestPoint_Pad_D1.5mm, symbol Connector:TestPoint
- added TP4: USB-, TestPoint:TestPoint_Pad_D1.5mm, symbol Connector:TestPoint
- added TP5: CHRG, TestPoint:TestPoint_Pad_D1.5mm, symbol Connector:TestPoint
- added TP6: STDBY, TestPoint:TestPoint_Pad_D1.5mm, symbol Connector:TestPoint
- added TP7: SRX, TestPoint:TestPoint_THTPad_D1.5mm_Drill0.7mm, symbol Connector:TestPoint
- added TP8: BAT, TestPoint:TestPoint_THTPad_D1.5mm_Drill0.7mm, symbol Connector:TestPoint
- added TP9: TEMP, TestPoint:TestPoint_Pad_D1.5mm, symbol Connector:TestPoint
- A1: footprint Module:RaspberryPi_Pico_W_SMD -> pico:RaspberryPi_Pico_W_SMD_THTdebug
- R2, R3: footprint (none) -> Resistor_SMD:R_0603_1608Metric_Pad0.98x0.95mm_HandSolder
- TP13: renamed from TP_KROW1; value TestPoint -> KROW1; footprint TestPoint:TestPoint_THTPad_D1.5mm_Drill0.7mm -> TestPoint:TestPoint_Pad_D1.0mm
- TP14: renamed from TP_VBUS; value VBUS test point -> VBUS
- TP15: renamed from TP_KROW2; value TestPoint -> KROW2; footprint TestPoint:TestPoint_THTPad_D1.5mm_Drill0.7mm -> TestPoint:TestPoint_Pad_D1.0mm
- TP16: renamed from TP_VSYS; value VSYS test point -> VSYS
- TP17: renamed from TP_3V3; value 3V3 test point -> 3V3
- TP18: renamed from TP_KROW3; value TestPoint -> KROW3; footprint TestPoint:TestPoint_THTPad_D1.5mm_Drill0.7mm -> TestPoint:TestPoint_Pad_D1.0mm
- TP19: renamed from TP_KROW4; value TestPoint -> KROW4; footprint TestPoint:TestPoint_THTPad_D1.5mm_Drill0.7mm -> TestPoint:TestPoint_Pad_D1.0mm
- TP20: renamed from TP_KROW5; value TestPoint -> KROW5; footprint TestPoint:TestPoint_THTPad_D1.5mm_Drill0.7mm -> TestPoint:TestPoint_Pad_D1.0mm
- TP21: renamed from TP_GND; value GND test point -> GND
- TP22: renamed from TP_KROW6; value TestPoint -> KROW6; footprint TestPoint:TestPoint_THTPad_D1.5mm_Drill0.7mm -> TestPoint:TestPoint_Pad_D1.0mm
- TP23: renamed from TP_KCOL1; value TestPoint -> KCOL1; footprint TestPoint:TestPoint_THTPad_D1.5mm_Drill0.7mm -> TestPoint:TestPoint_Pad_D1.0mm
- TP24: renamed from TP_KCOL2; value TestPoint -> KCOL2; footprint TestPoint:TestPoint_THTPad_D1.5mm_Drill0.7mm -> TestPoint:TestPoint_Pad_D1.0mm
- TP25: renamed from TP_KCOL3; value TestPoint -> KCOL3; footprint TestPoint:TestPoint_THTPad_D1.5mm_Drill0.7mm -> TestPoint:TestPoint_Pad_D1.0mm
- TP26: renamed from TP_KCOL4; value TestPoint -> KCOL4; footprint TestPoint:TestPoint_THTPad_D1.5mm_Drill0.7mm -> TestPoint:TestPoint_Pad_D1.0mm
- TP_LED1, TP_LED2: footprint TestPoint:TestPoint_THTPad_D1.5mm_Drill0.7mm -> TestPoint:TestPoint_Pad_D1.5mm
Connections:
- net +3V3: now also J3.3 (Pin_3), C22.1, C23.1, JP5.1 (A); no longer J3.1 (Pin_1), U2.6 (E3)
- net +5V: now also A1.40 (VBUS), C18.2, Q1.1 (G), Q2.1 (G), R1.1, TP14.1, C19.1, C20.1, C21.1, C24.1, D26.1 (K), F1.2, JP2.1 (A), R16.1, TP12.1
- net GND: now also C15.1, J3.1 (Pin_1), C19.2, C20.2, C21.2, C22.2, C23.2, C24.2, C25.2, JP3.1 (A), JP4.1 (A), R16.2; no longer C15.2, J3.3 (Pin_3), U2.4 (~{E1}), U2.5 (~{E2})
- net MAG_CLK: now also J4.4 (Pin_4); no longer J4.5 (Pin_5)
- net MAG_CSN: now also J4.3 (Pin_3); no longer J4.6 (Pin_6)
- net MAG_DO: now also J4.5 (Pin_5); no longer J4.4 (Pin_4)
- net MAG_OUT: now also J4.2 (Pin_2); no longer J4.7 (Pin_7)
- net MAG_PUSH: now also J4.1 (Pin_1); no longer J4.8 (Pin_8)
- net SRX: now also TP7.1
- net USB_D+: now also TP3.1
- net USB_D-: now also TP4.1
- net VBAT: now also TP10.1
- net at BT1.1 (+), C16.1, U4.C3 (BAT): now also TP8.1
- net at DB1.2 (A), R2.2: now also TP6.1
- net at R9.1, TH1.1, U1.1 (TEMP): now also TP9.1
- net at R13.1, U4.B3 (Vdd): now also C15.2; no longer C15.1
- net at DB2.2 (A), R3.2: now also TP5.1
- net at R14.2, R15.2, U5.3 (FB): now also TP11.1
- net at L1.2, U5.1 (SW): now also D25.2 (A)
- net BATT_5V renamed BAT_5V
- net BAT_5V: now also D25.1 (K), D26.2 (A), JP2.2 (B)
- removed net VBUS: A1.40 (VBUS), C18.2, J6.A4 (VBUS), J6.A9 (VBUS), J6.B4 (VBUS), J6.B9 (VBUS), Q1.1 (G), Q2.1 (G), R1.1, TP14.1
- net VSYS renamed BAT_VSYS
- net BAT_VSYS: now also C25.1
- new net: JP3.2 (B), U2.4 (~{E1})
- new net: JP4.2 (B), U2.5 (~{E2})
- new net: JP5.2 (B), U2.6 (E3)
- new net: F1.1, J6.A4 (VBUS), J6.A9 (VBUS), J6.B4 (VBUS), J6.B9 (VBUS)
Other:
- note added: "3.3V"
- note added: "5V"
- note added: "BAT_5V won't suffer from usb's voltage backfeeding i think"
- note added: "Is this necessary?"
- note added: "Maybe replace with schottky diodes instead? shave a couple bucks off ok while i have schottky, i dont think it would work with the boost converter"
- note added: "To make KiCad happy"
- note added: "cut jumper if schottky!"
- note added: "mosfet pulldown"
- note removed: "Maybe add a PPTC here. ~2A hold 3~4A trip should be okay"
- note removed: "Maybe replace with schottky diodes instead? shave a couple bucks off"
- note removed: "TODO: 5V source is a bit more complicated"
- note removed: "TODO: Schottky diode"
- note removed: "mosfet pulldown not required, builtin of the pico"
- moved on the sheet: A1, BT1, C13, C15, C16, C17, C3, J1, J2, L1, O1, Q1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

Commit message: everything routed except led
Parts:
- removed JP2: Batt 5v no schottky, Jumper:SolderJumper-2_P1.3mm_Bridged_Pad1.0x1.5mm, symbol Jumper:SolderJumper_2_Bridged
- added D27: SS54, Diode_SMD:D_SMA_Handsoldering, symbol Device:D_Schottky
- added Q3: AO3415, Package_TO_SOT_SMD:SOT-23_Handsoldering, symbol custom:AO3415
- D26: now fitted
- TP27: renamed from TP_LED1; value TestPoint -> LED1
- TP28: renamed from TP_LED2; value TestPoint -> LED2
Connections:
- net +3V3: now also J1.2 (Pin_2); no longer J1.1 (Pin_1)
- net +5V: now also J1.3 (Pin_3), D27.1 (K); no longer A1.40 (VBUS), C18.2, C21.1, F1.2, J1.2 (Pin_2), Q1.1 (G), Q2.1 (G), R1.1, R16.1, TP14.1
- net BAT_VSYS: now also Q1.3 (D); no longer Q1.2 (S)
- net GND: now also J1.1 (Pin_1), SW1.3 (C); no longer J1.3 (Pin_3)
- net MOTR_UH: now also A1.9 (GPIO6); no longer A1.15 (GPIO11)
- net MOTR_UL: now also A1.10 (GPIO7); no longer A1.14 (GPIO10)
- net MOTR_VH: now also A1.11 (GPIO8); no longer A1.12 (GPIO9)
- net MOTR_VL: now also A1.12 (GPIO9); no longer A1.11 (GPIO8)
- net MOTR_WH: now also A1.14 (GPIO10); no longer A1.10 (GPIO7)
- net MOTR_WL: now also A1.15 (GPIO11); no longer A1.9 (GPIO6)
- net MT_ROW1: now also U2.10 (Y5); no longer U2.15 (Y0)
- net MT_ROW2: now also U2.11 (Y4); no longer U2.14 (Y1)
- net MT_ROW3: now also U2.12 (Y3); no longer U2.13 (Y2)
- net MT_ROW4: now also U2.13 (Y2); no longer U2.12 (Y3)
- net MT_ROW5: now also U2.14 (Y1); no longer U2.11 (Y4)
- net MT_ROW6: now also U2.15 (Y0); no longer U2.10 (Y5)
- net SRX: now also SW1.1 (A), Q3.2 (S); no longer SW1.2 (B)
- net VBAT: now also Q1.2 (S), Q3.3 (D); no longer C14.2, Q1.3 (D), SW1.1 (A)
- net at DB2.1 (K), JP1.1 (A), U1.7 (~{CHRG}): now also TP5.1
- net at DB2.2 (A), R3.2: no longer TP5.1
- net at DB1.2 (A), R2.2: no longer TP6.1
- net at DB1.1 (K), U1.6 (~{STDBY}): now also TP6.1
- new net: C14.2, Q3.1 (G), SW1.2 (B)
- new net VBUS: A1.40 (VBUS), C18.2, C21.1, D27.2 (A), F1.2, Q1.1 (G), Q2.1 (G), R1.1, R16.1, TP14.1
- no-connect marks 46 -> 45
Other:
- note added: "5v on top!"
- note added: "BAT_5V won't suffer from usb's voltage backfeeding i think UPDATE: BUT usb 5v detect would! add diode on vbus side Im adding another schottky on batt since i have the parts anyways if its not needed, just bridge with solder"
- note removed: "BAT_5V won't suffer from usb's voltage backfeeding i think"
- note removed: "Same as dial board"
- note removed: "cut jumper if schottky!"
- moved on the sheet: Q1, SW1, TP10, TP5, TP6, TP7

Commit message: before ground pour
Parts:
- TP16: footprint TestPoint:TestPoint_THTPad_D1.5mm_Drill0.7mm -> TestPoint:TestPoint_Pad_D1.5mm
Changed lines of the file:
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@@
 			)
 		)
-		(property "Footprint" "TestPoint:TestPoint_THTPad_D1.5mm_Drill0.7mm"
+		(property "Footprint" "TestPoint:TestPoint_Pad_D1.5mm"
 			(at 123.19 184.15 0)
 			(hide yes)

Commit message: copper done todo: silkscreen + art
Parts:
- TP1, TP10, TP11, TP12, TP13, TP14, TP15, TP16, TP17, TP18, TP19, TP2, TP20, TP21, TP22, TP23, TP24, TP25, TP26, TP27, TP28, TP3, TP4, TP5, TP6, TP7, TP8, TP9: now left out of the parts list
Changed lines of the file:
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@@
 		(body_style 1)
 		(exclude_from_sim no)
-		(in_bom yes)
+		(in_bom no)
 		(on_board yes)
 		(in_pos_files yes)
@@
 		(body_style 1)
 		(exclude_from_sim no)
-		(in_bom yes)
+		(in_bom no)
 		(on_board yes)
 		(in_pos_files yes)
@@
 		(body_style 1)
 		(exclude_from_sim no)
-		(in_bom yes)
+		(in_bom no)
 		(on_board yes)
 		(in_pos_files yes)
@@
 		(body_style 1)
 		(exclude_from_sim no)
-		(in_bom yes)
+		(in_bom no)
 		(on_board yes)
 		(in_pos_files yes)
@@
 		(body_style 1)
 		(exclude_from_sim no)
-		(in_bom yes)
+		(in_bom no)
 		(on_board yes)
 		(in_pos_files yes)
@@
 		(body_style 1)
 		(exclude_from_sim no)
-		(in_bom yes)
+		(in_bom no)
 		(on_board yes)
 		(in_pos_files yes)
@@
 		(body_style 1)
 		(exclude_from_sim no)
-		(in_bom yes)
+		(in_bom no)
 		(on_board yes)
 		(in_pos_files yes)
@@
 		(body_style 1)
 		(exclude_from_sim no)
-		(in_bom yes)
+		(in_bom no)
 		(on_board yes)
 		(in_pos_files yes)
@@
 		(body_style 1)
 		(exclude_from_sim no)
-		(in_bom yes)
+		(in_bom no)
 		(on_board yes)
 		(in_pos_files yes)
@@
 		(body_style 1)
 		(exclude_from_sim no)
-		(in_bom yes)
+		(in_bom no)
 		(on_board yes)
 		(in_pos_files yes)
@@
 		(body_style 1)
 		(exclude_from_sim no)
-		(in_bom yes)
+		(in_bom no)
 		(on_board yes)
 		(in_pos_files yes)
@@
 		(body_style 1)
 		(exclude_from_sim no)
-		(in_bom yes)
+		(in_bom no)
 		(on_board yes)
 		(in_pos_files yes)
@@
 		(body_style 1)
 		(exclude_from_sim no)
-		(in_bom yes)
+		(in_bom no)
 		(on_board yes)
 		(in_pos_files yes)
@@
 		(body_style 1)
 		(exclude_from_sim no)
-		(in_bom yes)
+		(in_bom no)
 		(on_board yes)
 		(in_pos_files yes)
@@
 		(body_style 1)
 		(exclude_from_sim no)
-		(in_bom yes)
+		(in_bom no)
 		(on_board yes)
 		(in_pos_files yes)
@@
 		(body_style 1)
 		(exclude_from_sim no)
-		(in_bom yes)
+		(in_bom no)
 		(on_board yes)
 		(in_pos_files yes)
@@
 		(body_style 1)
 		(exclude_from_sim no)
-		(in_bom yes)
+		(in_bom no)
 		(on_board yes)
 		(in_pos_files yes)
@@
 		(body_style 1)
 		(exclude_from_sim no)
-		(in_bom yes)
+		(in_bom no)
 		(on_board yes)
 		(in_pos_files yes)
@@
 		(body_style 1)
 		(exclude_from_sim no)
-		(in_bom yes)
+		(in_bom no)
 		(on_board yes)
 		(in_pos_files yes)
@@
 		(body_style 1)
 		(exclude_from_sim no)
-		(in_bom yes)
+		(in_bom no)
 		(on_board yes)
 		(in_pos_files yes)
@@
 		(body_style 1)
 		(exclude_from_sim no)
-		(in_bom yes)
+		(in_bom no)
 		(on_board yes)
 		(in_pos_files yes)
@@
 		(body_style 1)
 		(exclude_from_sim no)
-		(in_bom yes)
+		(in_bom no)
 		(on_board yes)
 		(in_pos_files yes)
@@
 		(body_style 1)
 		(exclude_from_sim no)
-		(in_bom yes)
+		(in_bom no)
 		(on_board yes)
 		(in_pos_files yes)
@@
 		(body_style 1)
 		(exclude_from_sim no)
-		(in_bom yes)
+		(in_bom no)
 		(on_board yes)
 		(in_pos_files yes)
@@
 		(body_style 1)
 		(exclude_from_sim no)
-		(in_bom yes)
+		(in_bom no)
 		(on_board yes)
 		(in_pos_files yes)
@@
 		(body_style 1)
 		(exclude_from_sim no)
-		(in_bom yes)
+		(in_bom no)
 		(on_board yes)
 		(in_pos_files yes)
@@
 		(body_style 1)
 		(exclude_from_sim no)
-		(in_bom yes)
+		(in_bom no)
 		(on_board yes)
 		(in_pos_files yes)
@@
 		(body_style 1)
 		(exclude_from_sim no)
-		(in_bom yes)
+		(in_bom no)
 		(on_board yes)
 		(in_pos_files yes)

Commit message: 6-2-fab1
do not use! (changed via dimensions to fit jlc's free tier)
Parts:
- J1, J2: now not fitted; now left out of the parts list
- U1: footprint Package_SO:SOIC-8-1EP_3.9x4.9mm_P1.27mm_EP2.41x3.3mm_ThermalVias -> footprints:SOIC-8-1EP_3.9x4.9mm_P1.27mm_EP2.41x3.3mm_ThermalVias
Changed lines of the file:
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@@
 		(body_style 1)
 		(exclude_from_sim no)
-		(in_bom yes)
+		(in_bom no)
 		(on_board yes)
 		(in_pos_files yes)
-		(dnp no)
+		(dnp yes)
 		(fields_autoplaced yes)
 		(property "Reference" "J2"
@@
 			)
 		)
-		(property "Footprint" "Package_SO:SOIC-8-1EP_3.9x4.9mm_P1.27mm_EP2.41x3.3mm_ThermalVias"
+		(property "Footprint" "footprints:SOIC-8-1EP_3.9x4.9mm_P1.27mm_EP2.41x3.3mm_ThermalVias"
 			(at 76.708 93.98 0)
 			(hide yes)
@@
 		(body_style 1)
 		(exclude_from_sim no)
-		(in_bom yes)
+		(in_bom no)
 		(on_board yes)
 		(in_pos_files yes)
-		(dnp no)
+		(dnp yes)
 		(property "Reference" "J1"
 			(at 344.17 148.5901 0)
