File: PCB/blackmacro_dial/blackmacro_dial.kicad_sch (KiCad schematic)
At the start: 34 parts, among them J1 MagEncoderConn, J2 MotorControlConn, J3 MotorOutConn, J4 PowerConn, U1 MT6701CT, U2 TMC6300

Commit message: schematics done, working on pcb
Changed lines of the file:
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@@
 		)
 		(pin "8"
+			(alternate "~{CS}")
 		)
 		(pin "5"
 		)
 		(pin "7"
+			(alternate "CLK")
 		)
 		(pin "6"
+			(alternate "DO")
 		)
 		(instances
